File: hw/RGB_module.kicad_sch (KiCad schematic)
At the start: 11 parts, among them J1 Conn_01x04, J2 Conn_01x04, J3 Conn_01x03, U1 ZSCS-2016C-08D-Z4

Commit message: board_v2
Parts:
- removed H1, H2: MountingHole, MountingHole:MountingHole_3.2mm_M3_Pad_TopBottom, symbol Mechanical:MountingHole
- removed J3: Conn_01x03, Connector_PinHeader_2.54mm:PinHeader_1x03_P2.54mm_Vertical, symbol Connector_Generic:Conn_01x03
- added R3: 0, Resistor_SMD:R_0603_1608Metric_Pad0.98x0.95mm_HandSolder, symbol Device:R
- added R4: 100k, Resistor_SMD:R_0603_1608Metric_Pad0.98x0.95mm_HandSolder, symbol Device:R
- R1, R2: value 8 -> 33; footprint Resistor_SMD:R_0402_1005Metric -> Resistor_SMD:R_0603_1608Metric; LCSC C137928 -> C23140
Connections:
- net +3.3V: now also R4.2
- net GND: now also R3.1
- net at U1.4 (ADDR): now also R3.2, R4.1

Commit message: board_v3
Connections:
- net SCL: no longer names the net of J1.4 (Pin_4), J2.4 (Pin_4), U1.1 (SCL)
- net SDA: no longer names the net of J1.3 (Pin_3), J2.3 (Pin_3), U1.2 (SDA)
Other:
- moved on the sheet: C1, D1, D2, R1, R2, R3, R4
