File: hw/RGB_module.kicad_pcb (KiCad board)
At the start: 2 copper layers, 30 x 10 mm, 11 parts, among them J1 Conn_01x04, J2 Conn_01x04, J3 Conn_01x03, U1 ZSCS-2016C-08D-Z4

Commit message: board_v2
Parts:
- removed H1, H2: MountingHole, MountingHole:MountingHole_3.2mm_M3_Pad_TopBottom
- removed J3: Conn_01x03, Connector_PinHeader_2.54mm:PinHeader_1x03_P2.54mm_Vertical
- added R3: 0, Resistor_SMD:R_0603_1608Metric_Pad0.98x0.95mm_HandSolder, F.Cu at (45.1, 31.4)
- added R4: 100k, Resistor_SMD:R_0603_1608Metric_Pad0.98x0.95mm_HandSolder, F.Cu at (48.5, 31.4)
- R1, R2: value 8 -> 33; footprint Resistor_SMD:R_0402_1005Metric -> Resistor_SMD:R_0603_1608Metric
- moved C1 34.5 mm to (46.6, 26.5), turned to 0 degrees
- moved D1 32.8 mm to (44.3, 27.9)
- moved U1 32.6 mm to (46.8, 27.9), turned to 90 degrees
- moved R2 32.5 mm to (48.8, 31.1)
- moved D2 32.3 mm to (49.3, 27.9)
- moved R1 32.3 mm to (44.8, 31.1)
- moved J2 32.2 mm to (42.8, 27.9), turned to 0 degrees
- moved J1 29.9 mm to (50.8, 27.9), turned to 0 degrees
Routing:
- net +3.3V: track 20.9 -> 32.8 mm, vias 1 -> 2
- net SDA: track 7.12 -> 13.6 mm, vias 1 -> 2
- net Net-(U1-ADDR): track 8.44 -> 7.26 mm, vias 0 -> 1
- net SCL: track 12.6 -> 11.9 mm
- net GND: track 2.65 -> 2.01 mm, vias 19 -> 12
Other:
- outline, holes or cut-outs redrawn

Commit message: board_v3
Parts:
- R3, R4: moved to B.Cu
- moved R2 12.1 mm to (47.7, 19.0)
- moved R1 12.1 mm to (44.3, 19.0)
- moved J1 9.88 mm to (46.0, 19.3)
- moved R4 6.42 mm to (47.7, 25.0)
- moved R3 6.41 mm to (44.3, 25.0)
- moved C1 6.18 mm to (45.6, 20.4)
- moved D1 5.99 mm to (43.5, 22.0), turned to 90 degrees
- moved D2 5.99 mm to (48.5, 22.0), turned to 90 degrees
- moved U1 5.99 mm to (46.0, 22.0)
- moved J2 4.55 mm to (46.0, 24.7)
Connections:
- net SCL renamed Net-(J1-Pin_4)
- net SDA renamed Net-(J1-Pin_3)
Routing:
- net +3.3V: track 32.8 -> 19.7 mm, vias 2 -> 1
- net Net-(J1-Pin_3): track 13.6 -> 7.29 mm, vias 2 -> 1
- net Net-(J1-Pin_4): track 11.9 -> 6.91 mm
- net Net-(U1-ADDR): track 7.26 -> 5.06 mm, vias 1 -> 0
- net GND: track 2.01 -> 0.00 mm, vias 12 -> 11
Other:
- board size 30 x 10 mm -> 22 x 11 mm

Commit message: PCB_update
Parts:
- moved R3 1.00 mm to (44.3, 26.0)
- moved R4 1.00 mm to (47.7, 26.0)
Routing:
- net Net-(U1-ADDR): track 5.06 -> 7.06 mm
- net +3.3V: track 19.7 -> 20.8 mm
Other:
- outline, holes or cut-outs redrawn
Changed lines of the file:
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@@
 	(footprint "Resistor_SMD:R_0603_1608Metric_Pad0.98x0.95mm_HandSolder"
 		(layer "B.Cu")
-		(at 47.7 25)
+		(at 47.7 26)
 		(descr "Resistor SMD 0603 (1608 Metric), square (rectangular) end terminal, IPC_7351 nominal with elongated pad for handsoldering. (Body size source: IPC-SM-782 page 72, https://www.pcb-3d.com/wordpress/wp-content/uploads/ipc-sm-782a_amendment_1_and_2.pdf), generated with kicad-footprint-generator")
 		(tags "resistor handsolder")
 		(property "Reference" "R4"
-			(at 0 1.43 0)
+			(at 2.41 0 90)
 			(layer "B.SilkS")
 			(effects
@@
 	(footprint "Resistor_SMD:R_0603_1608Metric_Pad0.98x0.95mm_HandSolder"
 		(layer "B.Cu")
-		(at 44.3 25)
+		(at 44.3 26)
 		(descr "Resistor SMD 0603 (1608 Metric), square (rectangular) end terminal, IPC_7351 nominal with elongated pad for handsoldering. (Body size source: IPC-SM-782 page 72, https://www.pcb-3d.com/wordpress/wp-content/uploads/ipc-sm-782a_amendment_1_and_2.pdf), generated with kicad-footprint-generator")
 		(tags "resistor handsolder")
 		(property "Reference" "R3"
-			(at 0 1.43 180)
+			(at -2.33 0 270)
 			(layer "B.SilkS")
 			(effects
@@
 		(layer "Edge.Cuts")
 	)
-	(gr_rect
-		(start 35 16.5)
-		(end 57 27.5)
+	(gr_arc
+		(start 35 19.5)
+		(mid 35.87868 17.37868)
+		(end 38 16.5)
 		(stroke
-			(width 0.1)
-			(type solid)
-		)
-		(fill no)
+			(width 0.05)
+			(type default)
+		)
+		(layer "Edge.Cuts")
+	)
+	(gr_arc
+		(start 57 24.5)
+		(mid 56.12132 26.62132)
+		(end 54 27.5)
+		(stroke
+			(width 0.05)
+			(type default)
+		)
+		(layer "Edge.Cuts")
+	)
+	(gr_line
+		(start 57 24.5)
+		(end 57 19.5)
+		(stroke
+			(width 0.05)
+			(type default)
+		)
+		(layer "Edge.Cuts")
+	)
+	(gr_arc
+		(start 54 16.5)
+		(mid 56.12132 17.37868)
+		(end 57 19.5)
+		(stroke
+			(width 0.05)
+			(type default)
+		)
+		(layer "Edge.Cuts")
+	)
+	(gr_line
+		(start 38 27.5)
+		(end 54 27.5)
+		(stroke
+			(width 0.05)
+			(type default)
+		)
+		(layer "Edge.Cuts")
+	)
+	(gr_line
+		(start 54 16.5)
+		(end 38 16.5)
+		(stroke
+			(width 0.05)
+			(type default)
+		)
 		(layer "Edge.Cuts")
 	)
@@
 		)
 		(fill no)
+		(layer "Edge.Cuts")
+	)
+	(gr_arc
+		(start 38 27.5)
+		(mid 35.87868 26.62132)
+		(end 35 24.5)
+		(stroke
+			(width 0.05)
+			(type default)
+		)
+		(layer "Edge.Cuts")
+	)
+	(gr_line
+		(start 35 19.5)
+		(end 35 24.5)
+		(stroke
+			(width 0.05)
+			(type default)
+		)
 		(layer "Edge.Cuts")
 	)
@@
 	)
 	(via
-		(at 36.449 26.2636)
+		(at 37 26)
 		(size 0.6)
 		(drill 0.3)
@@
 	)
 	(via
-		(at 55.9054 17.907)
+		(at 55 18)
 		(size 0.6)
 		(drill 0.3)
@@
 	)
 	(via
-		(at 55.8292 26.2636)
+		(at 55 26)
 		(size 0.6)
 		(drill 0.3)
@@
 	)
 	(via
-		(at 43.0022 26.416)
+		(at 41.75 25.97)
 		(size 0.6)
 		(drill 0.3)
@@
 	)
 	(segment
-		(start 44.45 22.7584)
+		(start 44.31 22.8984)
 		(end 45.5 21.7084)
+		(width 0.3)
+		(layer "F.Cu")
+		(net 2)
+	)
+	(segment
+		(start 45.5 21.7084)
+		(end 45.5 20.625)
 		(width 0.3)
 		(layer "F.Cu")
@@
 	)
 	(segment
-		(start 45.5 21.7084)
-		(end 45.5 20.625)
+		(start 44.31 23.6344)
+		(end 44.31 22.8984)
 		(width 0.3)
 		(layer "F.Cu")
@@
 	)
 	(segment
-		(start 44.45 23.7744)
-		(end 44.45 22.7584)
-		(width 0.3)
-		(layer "F.Cu")
-		(net 2)
-	)
-	(segment
 		(start 44.6405 23.9649)
-		(end 44.45 23.7744)
+		(end 44.31 23.6344)
 		(width 0.3)
 		(layer "F.Cu")
@@
 	)
 	(segment
-		(start 44.323 25.436846)
-		(end 44.712154 25.826)
-		(width 0.3)
-		(layer "B.Cu")
-		(net 2)
-	)
-	(segment
 		(start 45.141 20.8078)
 		(end 45.32 20.9868)
@@
 	)
 	(segment
+		(start 44.311 26.46)
+		(end 44.677 26.826)
+		(width 0.3)
+		(layer "B.Cu")
+		(net 2)
+	)
+	(segment
 		(start 45.148 19)
 		(end 45.148 20.3892)
@@
 	)
 	(segment
-		(start 44.712154 25.826)
-		(end 47.7865 25.826)
-		(width 0.3)
-		(layer "B.Cu")
-		(net 2)
-	)
-	(segment
 		(start 45.148 20.3892)
 		(end 45.141 20.3962)
@@
 	)
 	(segment
-		(start 47.7865 25.826)
-		(end 48.6125 25)
-		(width 0.3)
-		(layer "B.Cu")
-		(net 2)
-	)
-	(segment
-		(start 44.323 24.2824)
-		(end 44.6405 23.9649)
-		(width 0.3)
-		(layer "B.Cu")
-		(net 2)
-	)
-	(segment
-		(start 44.323 25.436846)
-		(end 44.323 24.2824)
+		(start 44.311 24.2944)
+		(end 44.311 26.46)
+		(width 0.3)
+		(layer "B.Cu")
+		(net 2)
+	)
+	(segment
+		(start 44.6405 23.9649)
+		(end 44.311 24.2944)
+		(width 0.3)
+		(layer "B.Cu")
+		(net 2)
+	)
+	(segment
+		(start 44.677 26.826)
+		(end 47.7865 26.826)
+		(width 0.3)
+		(layer "B.Cu")
+		(net 2)
+	)
+	(segment
+		(start 47.7865 26.826)
+		(end 48.6125 26)
 		(width 0.3)
 		(layer "B.Cu")
@@
 	)
 	(segment
+		(start 46.7875 26)
+		(end 46.7875 25)
+		(width 0.2)
+		(layer "B.Cu")
+		(net 7)
+	)
+	(segment
+		(start 46.7875 25)
+		(end 46 24.2125)
+		(width 0.2)
+		(layer "B.Cu")
+		(net 7)
+	)
+	(segment
 		(start 45.2125 25)
 		(end 46 24.2125)
@@
 	)
 	(segment
-		(start 46.7875 25)
-		(end 46 24.2125)
+		(start 45.2125 26)
+		(end 45.2125 25)
 		(width 0.2)
 		(layer "B.Cu")
